File: SCHEMATICS/Matrix+RFID/Matrix+RFID.kicad_sch (KiCad schematic)
At the start: 13 parts, among them M1 SG90, SW1 Button, SW2 Push, U1 ESP32-WROOM-32, U3 BUCK 9V to 5V

Commit message: Matrix+RFID v2
Parts:
- added D3: LED, symbol Device:LED
- added R3: R, symbol Device:R
Connections:
- net 5V: now also R3.1
- net GND: now also D3.1 (K)
- new net: D3.2 (A), R3.2
Other:
- note added: "20/12/23"
- note added: "Strongbox v2"
- note removed: "6/12/23"
- note removed: "Strongbox v1"
- moved on the sheet: 9V
